File: pcb/Lily58.kicad_pcb (KiCad board)
At the start: 2 copper layers, 142.5 x 106.3 mm, 123 parts, among them J1 LED, J2 4PIN, P1 i2c_pin, P2 i2c_pin, P3 ICSP, P4 OLED, SW1 SW_PUSH, SW10 SW_PUSH, SW11 SW_PUSH, SW12 SW_PUSH, SW13 SW_PUSH, SW14 SW_PUSH, SW15 SW_PUSH, SW16 SW_PUSH, SW17 SW_PUSH, SW18 SW_PUSH, SW19 SW_PUSH, SW2 SW_PUSH, SW20 SW_PUSH, SW21 SW_PUSH, SW22 SW_PUSH, SW23 SW_PUSH, SW24 SW_PUSH, SW25 SW_PUSH, SW26 SW_PUSH, SW27 SW_PUSH, SW28 SW_PUSH, SW29 SW_PUSH, SW3 SW_PUSH, SW4 SW_PUSH, SW5 SW_PUSH, SW6 SW_PUSH, SW7 SW_PUSH, SW8 SW_PUSH, SW9 SW_PUSH, U1 ProMicro

Commit message: added name + case file
added name
Parts:
- moved G*** 4.40 mm to (101.4, 81.1) (x2)
Other:
- board text added: "Ananya Kirti"
- board text added: "Lily58"
- board text removed: "Lily58 × qtkb"
